File: pcb/motor_control_board/Hardware/Motorsteuerung_v3.sch (EAGLE design)
At the start: 74 parts, among them IC1 TMC5160-TA, IC2 CP2104, J4 10118193-0001LF, Q1 AO4882", Q2 AO4882", Q3 AO4882", Q4 AO4882", Q5 BC817, Q6 BC817, SW1 TL3342F160QG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

Commit message: Production Files
Other:
- note added: "3V3 to 5V Converter"
- note added: "Neopixel LED with level shifter"
- moved on the sheet: C23, C24, C25, C26, D3, J4, U2, U4
