File: pcb/end_effector_board/PCB/42mm_Erweiterungsplatine.brd (EAGLE design)
At the start: 42 x 42 mm, 68 parts, among them IC2 CP2104, J4 10118193-0001LF, Q5 BC817, Q6 BC817, SW1 KMR2, SW3 KMR2, U1 SN65HVD232, U2 ESP32-PICO-D4, U3 TPSM53603RDAR, U4 74LVC1G08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

Commit message: Replaced Level Shifter for LEDs. Thanks to Yu-Lien Fang for noticing!
Parts:
- U4, U5: value 74LVC1G08 -> 74HCT1G08
Changed lines of the file:
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@@
 </layers>
 <board>
-<fusionsync huburn="a.cGVyc29uYWw6dWUyYjBjZmRm" projecturn="a.cGVyc29uYWw6dWUyYjBjZmRmIzIwMTkwNzEwMjAzMDM3MDUx" f3durn="urn:adsk.wipprod:dm.lineage:HVTAxYjFStKtDTsvKg0P5A" pcbguid="" lastpulledtime="" lastsyncedchangeguid="a4446e10-05e5-533a-4639-39e679d7ad28" latestrevisionid="8cc320fa-5a1c-463b-bc90-c890698ea3c0" lastsyncedrevisionid="8cc320fa-5a1c-463b-bc90-c890698ea3c0" lastboardhashguid="d7b8679d-6363-d1fa-a133-b9b1690b6bac" lastpushedtime="2021-05-02T17:58:24Z" linktopcb3d="true"/>
+<fusionsync huburn="a.cGVyc29uYWw6dWUyYjBjZmRm" projecturn="a.cGVyc29uYWw6dWUyYjBjZmRmIzIwMTkwNzEwMjAzMDM3MDUx" f3durn="urn:adsk.wipprod:dm.lineage:HVTAxYjFStKtDTsvKg0P5A" pcbguid="" lastpulledtime="" lastsyncedchangeguid="a4446e10-05e5-533a-4639-39e679d7ad28" latestrevisionid="8cc320fa-5a1c-463b-bc90-c890698ea3c0" lastsyncedrevisionid="8cc320fa-5a1c-463b-bc90-c890698ea3c0" lastboardhashguid="d7b8679d-6363-d1fa-a133-b9b1690b6bac" lastpushedtime="2021-05-02T17:58:24Z" linktopcb3d="false"/>
 <plain>
 <wire x1="1.2" y1="0" x2="40.8" y2="0" width="0" layer="20"/>
@@
 <attribute name="VALUE" x="22.987" y="33.909" size="1.27" layer="27" rot="R180"/>
 </element>
-<element name="U4" library="74LVC1G00GW" package="SOT65P210X110-5N" override_package3d_urn="urn:adsk.eagle:package:21263399/2" override_package_urn="urn:adsk.eagle:footprint:21263400/1" value="74LVC1G08" x="16.891" y="28.956" smashed="yes">
+<element name="U4" library="74LVC1G00GW" package="SOT65P210X110-5N" override_package3d_urn="urn:adsk.eagle:package:21263399/2" override_package_urn="urn:adsk.eagle:footprint:21263400/1" value="74HCT1G08" x="16.891" y="28.956" smashed="yes">
 <attribute name="AVAILABILITY" value="Unavailable" x="16.891" y="28.956" size="1.778" layer="27" display="off"/>
 <attribute name="DESCRIPTION" value=" NAND Gate 1-Element 2-IN CMOS 5-Pin TSSOP T/R " x="16.891" y="28.956" size="1.778" layer="27" display="off"/>
@@
 <attribute name="VALUE" x="13.4333" y="24.506759375" size="2.084790625" layer="27" ratio="10" rot="SR0"/>
 </element>
-<element name="U5" library="74LVC1G00GW" package="SOT65P210X110-5N" override_package3d_urn="urn:adsk.eagle:package:21263399/2" override_package_urn="urn:adsk.eagle:footprint:21263400/1" value="74LVC1G08" x="16.891" y="24.384" smashed="yes">
+<element name="U5" library="74LVC1G00GW" package="SOT65P210X110-5N" override_package3d_urn="urn:adsk.eagle:package:21263399/2" override_package_urn="urn:adsk.eagle:footprint:21263400/1" value="74HCT1G08" x="16.891" y="24.384" smashed="yes">
 <attribute name="AVAILABILITY" value="Unavailable" x="16.891" y="24.384" size="1.778" layer="27" display="off"/>
 <attribute name="DESCRIPTION" value=" NAND Gate 1-Element 2-IN CMOS 5-Pin TSSOP T/R " x="16.891" y="24.384" size="1.778" layer="27" display="off"/>
