File: pcb/end_effector_board/PCB/42mm_Erweiterungsplatine.sch (EAGLE design)
At the start: 64 parts, among them IC2 CP2104, J4 10118193-0001LF, Q5 BC817, Q6 BC817, SW1 KMR2, SW3 KMR2, U1 SN65HVD232, U2 ESP32-PICO-D4, U3 TPSM53603RDAR, U4 74LVC1G08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

Commit message: Replaced Level Shifter for LEDs. Thanks to Yu-Lien Fang for noticing!
Parts:
- U4, U5: value 74LVC1G08 -> 74HCT1G08
Changed lines of the file:
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@@
 <part name="R9" library="rcl" library_urn="urn:adsk.eagle:library:334" deviceset="R-EU_" device="R0805" package3d_urn="urn:adsk.eagle:package:23553/2" value="10k"/>
 <part name="U$35" library="microbuilder" deviceset="3.3V" device="" value="+3V3"/>
-<part name="U4" library="74LVC1G00GW" deviceset="74LVC1G00GW" device="" override_package3d_urn="urn:adsk.eagle:package:21263399/2" override_package_urn="urn:adsk.eagle:footprint:21263400/1" value="74LVC1G08"/>
+<part name="U4" library="74LVC1G00GW" deviceset="74LVC1G00GW" device="" override_package3d_urn="urn:adsk.eagle:package:21263399/2" override_package_urn="urn:adsk.eagle:footprint:21263400/1" value="74HCT1G08"/>
 <part name="U$36" library="microbuilder" deviceset="GND" device=""/>
-<part name="U5" library="74LVC1G00GW" deviceset="74LVC1G00GW" device="" override_package3d_urn="urn:adsk.eagle:package:21263399/2" override_package_urn="urn:adsk.eagle:footprint:21263400/1" value="74LVC1G08"/>
+<part name="U5" library="74LVC1G00GW" deviceset="74LVC1G00GW" device="" override_package3d_urn="urn:adsk.eagle:package:21263399/2" override_package_urn="urn:adsk.eagle:footprint:21263400/1" value="74HCT1G08"/>
 <part name="U$37" library="microbuilder" deviceset="GND" device=""/>
 <part name="C5" library="rcl" library_urn="urn:adsk.eagle:library:334" deviceset="C-EU" device="C0805" package3d_urn="urn:adsk.eagle:package:23617/2" value="100n"/>
