File: pcb/motor_control_board/PCB/Motorsteuerung_v3.brd (EAGLE design)
At the start: 42 x 42 mm, 78 parts, among them IC1 TMC5160-TA, IC2 CP2104, J4 10118193-0001LF, Q1 AO4882", Q2 AO4882", Q3 AO4882", Q4 AO4882", Q5 BC817, Q6 BC817, SW1 TL3342F160QG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

Commit message: Replaced Level Shifter for LEDs. Thanks to Yu-Lien Fang for noticing!
Parts:
- U4: value 74LVC1G08 -> 74HCT1G08
Changed lines of the file:
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@@
 <?xml version="1.0" encoding="utf-8"?>
 <!DOCTYPE eagle SYSTEM "eagle.dtd">
-<eagle version="9.6.0">
+<eagle version="9.6.2">
 <drawing>
 <settings>
@@
 </layers>
 <board>
-<fusionsync huburn="a.cGVyc29uYWw6dWUyYjBjZmRm" projecturn="a.cGVyc29uYWw6dWUyYjBjZmRmIzIwMTkwNzEwMjAzMDM3MDUx" f3durn="urn:adsk.wipprod:dm.lineage:UkR34FPES4C5YuISfHm_-Q" pcbguid="9584afbd-31c7-4aba-ace3-9ba1bc9fa79f" lastpulledtime="" lastsyncedchangeguid="a4446e10-05e5-533a-4639-39e679d7ad28" latestrevisionid="" lastsyncedrevisionid="" lastboardhashguid="" lastpushedtime="" linktopcb3d="%12"/>
+<fusionsync huburn="a.cGVyc29uYWw6dWUyYjBjZmRm" projecturn="a.cGVyc29uYWw6dWUyYjBjZmRmIzIwMTkwNzEwMjAzMDM3MDUx" f3durn="urn:adsk.wipprod:dm.lineage:UkR34FPES4C5YuISfHm_-Q" pcbguid="9584afbd-31c7-4aba-ace3-9ba1bc9fa79f" lastpulledtime="" lastsyncedchangeguid="a4446e10-05e5-533a-4639-39e679d7ad28" latestrevisionid="" lastsyncedrevisionid="" lastboardhashguid="" lastpushedtime="" linktopcb3d="false"/>
 <plain>
 <rectangle x1="28.2" y1="20.7" x2="33.2" y2="25.7" layer="1"/>
@@
 <attribute name="VALUE" x="14.14" y="32.87" size="1.27" layer="28" rot="MR270"/>
 </element>
-<element name="U4" library="74LVC1G00GW" package="SOT65P210X110-5N" override_package3d_urn="urn:adsk.eagle:package:21263399/2" override_package_urn="urn:adsk.eagle:footprint:21263400/1" value="74LVC1G08" x="9.4" y="31.65" smashed="yes" rot="MR90">
+<element name="U4" library="74LVC1G00GW" package="SOT65P210X110-5N" override_package3d_urn="urn:adsk.eagle:package:21263399/2" override_package_urn="urn:adsk.eagle:footprint:21263400/1" value="74HCT1G08" x="9.4" y="31.65" smashed="yes" rot="MR90">
 <attribute name="AVAILABILITY" value="Unavailable" x="9.4" y="31.65" size="1.778" layer="28" rot="MR90" display="off"/>
 <attribute name="DESCRIPTION" value=" NAND Gate 1-Element 2-IN CMOS 5-Pin TSSOP T/R " x="9.4" y="31.65" size="1.778" layer="28" rot="MR90" display="off"/>
